File: src/rigidkey.kicad_pcb (KiCad board)
At the start: 2 copper layers, 50.8 x 19 mm, 21 parts, among them J1 Conn_01x04_Male, J2 USB_A, U1 STM32F103TB, U2 LP2985-33, U3 NUF2221W1, X1 12MHz

Commit message: Generate gerbers
Changed lines of the file:
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@@
   )
   (layers
-    (0 F.Cu signal hide)
-    (31 B.Cu signal hide)
-    (32 B.Adhes user hide)
-    (33 F.Adhes user hide)
-    (34 B.Paste user hide)
-    (35 F.Paste user hide)
-    (36 B.SilkS user hide)
+    (0 F.Cu signal)
+    (31 B.Cu signal)
+    (32 B.Adhes user)
+    (33 F.Adhes user)
+    (34 B.Paste user)
+    (35 F.Paste user)
+    (36 B.SilkS user)
     (37 F.SilkS user)
-    (38 B.Mask user hide)
+    (38 B.Mask user)
     (39 F.Mask user)
-    (40 Dwgs.User user hide)
-    (41 Cmts.User user hide)
-    (42 Eco1.User user hide)
-    (43 Eco2.User user hide)
+    (40 Dwgs.User user)
+    (41 Cmts.User user)
+    (42 Eco1.User user)
+    (43 Eco2.User user)
     (44 Edge.Cuts user)
     (45 Margin user)
-    (46 B.CrtYd user hide)
-    (47 F.CrtYd user hide)
-    (48 B.Fab user hide)
-    (49 F.Fab user hide)
+    (46 B.CrtYd user)
+    (47 F.CrtYd user)
+    (48 B.Fab user)
+    (49 F.Fab user)
   )
   (setup
@@
     (visible_elements FFFFFF7F)
     (pcbplotparams
-      (layerselection 0x010fc_ffffffff)
-      (usegerberextensions false)
+      (layerselection 0x010f0_ffffffff)
+      (usegerberextensions true)
       (usegerberattributes false)
       (usegerberadvancedattributes false)
@@
       (psa4output false)
       (plotreference true)
-      (plotvalue true)
+      (plotvalue false)
       (plotinvisibletext false)
       (padsonsilk false)
@@
       (outputformat 1)
       (mirror false)
-      (drillshape 1)
+      (drillshape 0)
       (scaleselection 1)
-      (outputdirectory ""))
+      (outputdirectory "gerbers/"))
   )
   (net 0 "")
@@
       (net 2 GND) (clearance 0.07874))
   )
-  (gr_text www.studio0xf.com (at 142.24 121.158) (layer F.SilkS)
+  (gr_text www.studio0xf.com (at 145.1356 122.9614) (layer F.SilkS)
     (effects (font (size 0.484 0.484) (thickness 0.0702)))
   )
-  (gr_text "Studio0xf\nRigidkey Rev. V01" (at 142.24 119.38) (layer F.SilkS)
+  (gr_text "Studio0xf\nRigidkey Rev. V01" (at 145.1356 121.1834) (layer F.SilkS)
     (effects (font (size 0.484 0.484) (thickness 0.0575)))
   )
