File: src/rigidkey.sch (KiCad schematic (older format))
At the start: 19 parts

Commit message: Create net list
Parts:
- removed C?: C, symbol Device:C
- removed R?: 100, symbol Device:R
- added C3, C4: 0.1uF, digikey-footprints:1206, symbol Device:C
- added D1: GREEN, digikey-footprints:1206, symbol Device:LED
- added R1: R, digikey-footprints:1206, symbol Device:R
- C1, C10, C2, C5, C6, C7, C8, C9: renamed from C?; footprint (none) -> digikey-footprints:1206
- J1: renamed from J?; footprint (none) -> digikey-footprints:PinHeader_1x4_P2.54mm_Drill1.02mm
- J2: renamed from J?; footprint (none) -> digikey-footprints:USB_Male_A_UP2-AH-1-TH
- JP1: renamed from JP?; footprint (none) -> digikey-footprints:PinHeader_1x2_P2.54mm_Drill1.02mm
- R2, R3: renamed from R?; footprint (none) -> digikey-footprints:1206
- U1: renamed from U?; footprint (none) -> FST:QFN36
- U2, U3: renamed from U?; footprint (none) -> FST:SOT23-5
- X1: renamed from X?; footprint (none) -> FST:ABM8G
Connections:
- net +3V3: now also U1.6 (VDDA), C4.1
- net BOOTO: now also U1.35 (BOOT0)
- net GND: now also J2.5 (Shield), U1.5 (VSSA), C3.2, C4.2, D1.1 (K)
- net at U1.15 (PB0): now also R1.1
- net at U1.4 (NRST): now also C3.1
- net USB_EN: no longer names the net of U1.29 (PA15)
- new net: D1.2 (A), R1.2
- no-connect marks 0 -> 18

Commit message: Layout board
Parts:
- J2: footprint digikey-footprints:USB_Male_A_UP2-AH-1-TH -> FST:USB_Male_A_UP2-AH-1-TH
- U3: footprint FST:SOT23-5 -> FST:SOT363
Connections:
- net -: now reaches U1.23 (USB_DM), U3.3 (D2i)
- net -: now also J2.2 (D-), U3.4 (D2c)
- net +: now reaches U1.24 (USB_DP), U3.1 (D1i)
- net +: now also J2.3 (D+), U3.6 (D1c)
Changed lines of the file:
@@
 F 0 "U3" H 8850 4020 70  0000 C CNN
 F 1 "NUF2221W1" H 8850 3899 70  0000 C CNN
-F 2 "FST:SOT23-5" H 8850 3650 50  0001 C CNN
+F 2 "FST:SOT363" H 8850 3650 50  0001 C CNN
 F 3 "" H 8850 3650 50  0001 C CNN
 	1    8850 3650
@@
 F 0 "J2" H 9820 3448 50  0000 R CNN
 F 1 "USB_A" H 9820 3539 50  0000 R CNN
-F 2 "digikey-footprints:USB_Male_A_UP2-AH-1-TH" H 10200 3500 50  0001 C CNN
+F 2 "FST:USB_Male_A_UP2-AH-1-TH" H 10200 3500 50  0001 C CNN
 F 3 " ~" H 10200 3500 50  0001 C CNN
 	1    10050 3550
@@
 Wire Wire Line
 	5250 5700 5250 5800
+Text Label 9550 3450 0    50   ~ 0
+-
+Text Label 9550 3550 0    50   ~ 0
++
+Text Label 7550 3550 0    50   ~ 0
++
+Text Label 7550 3650 0    50   ~ 0
+-
 $EndSCHEMATC

Commit message: Generate gerbers
Parts:
- R1: value R -> 500
Changed lines of the file:
@@
 P 5750 5450
 F 0 "R1" H 5820 5496 50  0000 L CNN
-F 1 "R" H 5820 5405 50  0000 L CNN
+F 1 "500" H 5820 5405 50  0000 L CNN
 F 2 "digikey-footprints:1206" V 5680 5450 50  0001 C CNN
 F 3 "~" H 5750 5450 50  0001 C CNN
